Commit message: head, wheel config

File: tr1_description/urdf/head/head.urdf.xacro (robot description, xacro)
@@ -80,5 +80,5 @@
 		<origin xyz="0 0 0.035"/>
     <axis xyz="0 0 1"/>
-		<limit effort="1.0" lower="-3.1415" upper="3.1415" velocity="0.5"/>
+		<limit effort="1.0" lower="-1.5708" upper="1.5708" velocity="0.5"/>
     <dynamics damping="0.1" friction="0.1"/>
 	</joint>
@@ -88,5 +88,5 @@
 		<origin xyz="0 0.090789 0.09"/>
     <axis xyz="1 0 0"/>
-		<limit effort="1.0" lower="-0.9" upper="0.4" velocity="0.5"/>
+		<limit effort="1.0" lower="-0.75" upper="0.4" velocity="0.5"/>
     <dynamics damping="0.1" friction="0.1"/>
 	</joint>
